File: Shifty-LED-Board/Shift-LED-Board.kicad_pcb (KiCad board)
At the start: 4 copper layers, 80 x 34 mm, 64 parts, among them U1 74AHCT595, U2 74AHCT595, U3 74AHCT595

Commit message: changed led resistors to 200ohm
Parts:
- R1, R10, R11, R12, R13, R14, R15, R16, R17, R18, R19, R2, R20, R21, R22, R23, R24, R3, R4, R5, R6, R7, R8, R9: value 270 -> 200
- R25, R26, R27: value 1k -> 10k
